Commit message: Adds flexible radius and tunes the finsler energies.

File: examples/albert_polluted_2.urdf (robot description, URDF)
Before this commit: robot albert_description, 45 links, 44 joints
Links:
- added link panda_vacuum_2
Joints:
- added joint panda_vacuum_joint_2: type fixed, parent panda_hand, child panda_vacuum_2, origin xyz=0 0 0.25 rpy=0 0 0
