Commit message: ft[esdf]: Makes collision links and self_collision_pairs optional in set_components.

File: examples/planar_urdf_2_joints.urdf (robot description, URDF)
Before this commit: robot panda_description, 5 links, 4 joints
Links:
- link panda_link4: geometry collision sphere radius=0.1; visual sphere radius=0.1
