Commit message: ft[rotation]: Changes panda examples to not use subgoal attribute angle anymore.

File: examples/panda_vacuum.urdf (robot description, URDF)
Before this commit: robot panda, 12 links, 11 joints
Links:
- removed link vacuum1_link
- removed link vacuum2_link
- added link vacuum_link, mass 0.00; collision cylinder length=0.02 radius=0.02; visual cylinder length=0.02 radius=0.02
Joints:
- removed joint panda_vacuum1_joint
- removed joint panda_vacuum2_joint
- added joint panda_vacuum_joint: type fixed, parent panda_link7, child vacuum_link, origin xyz=0.0 0 0.37 rpy=0 0 0
