Commit message: [ft_base_prismatic]: prismatic joint done

File: examples/panda_vacuum_base.urdf (robot description, URDF)
Before this commit: robot panda, 12 links, 11 joints
Links:
- added link base_link
Joints:
- added joint panda_joint_world: type fixed, parent world, child base_link, origin xyz=0 0 0 rpy=0 0 0
- joint mobile_joint_x: parent world -> base_link
