Commit message: kuka_iiwa_with_orientation.py added as example where orientation control is achieved on top of position control.

File: examples/iiwa7.urdf (robot description, URDF)
Before this commit: robot iiwa7, 10 links, 9 joints
Links:
- added link iiwa_link_ee_x; visual sphere radius=0.01
Joints:
- added joint iiwa_joint_ee_x: type fixed, parent iiwa_link_7, child iiwa_link_ee_x, origin xyz=0.045 0. 0. rpy=0 0 0
- joint iiwa_joint_ee: origin xyz=0 0 0.045 rpy=0 0 0 -> xyz=-0.045 0 0.045 rpy=0 0 0; parent iiwa_link_7 -> iiwa_link_ee_x
