Commit message: change of the order of the joints as per tomas changes

File: examples/dingo_kinova/urdf/dingo_kinova.urdf (robot description, URDF)
Before this commit: robot dingo_kinova, 26 links, 25 joints
Links:
- link arm_arm_link: geometry collision mesh filename=meshes/kinova/arm_link.STL; visual mesh filename=meshes/kinova/arm_link.STL
- link arm_base_link: geometry collision mesh filename=meshes/kinova/base_link.STL; visual mesh filename=meshes/kinova/base_link.STL
- link arm_forearm_link: geometry collision mesh filename=meshes/kinova/forearm_link.STL; visual mesh filename=meshes/kinova/forearm_link.STL
- link arm_lower_wrist_link: geometry collision mesh filename=meshes/kinova/lower_wrist_link.STL; visual mesh filename=meshes/kinova/lower_wrist_link.STL
- link arm_shoulder_link: geometry collision mesh filename=meshes/kinova/shoulder_link.STL; visual mesh filename=meshes/kinova/shoulder_link.STL
- link arm_upper_wrist_link: geometry collision mesh filename=meshes/kinova/upper_wrist_link.STL; visual mesh filename=meshes/kinova/upper_wrist_link.STL
- link chassis_link: geometry collision mesh filename=meshes/base/omni_chassis_collision.stl; visual mesh filename=meshes/base/omni_chassis_collision.stl
